File: level_shifters.kicad_sch (KiCad schematic)
At the start: 8 parts, among them IC1 TXU0101DBVR, IC2 TXU0101DBVR, IC3 TXU0101DBVR, IC4 TXU0101DBVR, IC5 TXU0101DBVR, IC6 TXU0101DBVR, IC7 TXU0101DBVR, IC8 TXU0101DBVR

Commit message: saving progress
Other:
- note added: "FanSenseShifter"
- note added: "PumpSenseShifter"
- note added: "ValveSense1Shifter"
- note added: "ValveSense2Shifter"
- note removed: "PumpSeneShifter"
Changed lines of the file:
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@@
 		)
 	)
-	(text "PumpSeneShifter"
+	(text "ValveSense1Shifter"
 		(exclude_from_sim no)
-		(at 27.94 82.804 0)
+		(at 28.956 82.804 0)
 		(effects
 			(font
@@
 		)
 	)
-	(text "PumpSeneShifter"
+	(text "ValveSense2Shifter"
 		(exclude_from_sim no)
-		(at 27.94 114.554 0)
+		(at 28.702 114.554 0)
 		(effects
 			(font
@@
 		)
 	)
-	(text "PumpSeneShifter"
+	(text "PumpSenseShifter"
 		(exclude_from_sim no)
 		(at 27.94 19.304 0)
@@
 		(effects
 			(font
+				(size 1.27 1.27)
+			)
+		)
+	)
+	(text "FanSenseShifter"
+		(exclude_from_sim no)
+		(at 27.686 51.054 0)
+		(effects
+			(font

Commit message: Prepped for production.
Parts:
- IC1, IC2, IC3, IC4, IC5, IC6, IC7, IC8: now not fitted; now left out of the parts list
Changed lines of the file:
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@@
 		(unit 1)
 		(exclude_from_sim no)
-		(in_bom yes)
-		(on_board yes)
-		(dnp no)
+		(in_bom no)
+		(on_board yes)
+		(dnp yes)
 		(fields_autoplaced yes)
 		(property "Reference" "IC6"
@@
 		(unit 1)
 		(exclude_from_sim no)
-		(in_bom yes)
-		(on_board yes)
-		(dnp no)
+		(in_bom no)
+		(on_board yes)
+		(dnp yes)
 		(fields_autoplaced yes)
 		(property "Reference" "IC5"
@@
 		(unit 1)
 		(exclude_from_sim no)
-		(in_bom yes)
-		(on_board yes)
-		(dnp no)
+		(in_bom no)
+		(on_board yes)
+		(dnp yes)
 		(fields_autoplaced yes)
 		(property "Reference" "IC7"
@@
 		(unit 1)
 		(exclude_from_sim no)
-		(in_bom yes)
-		(on_board yes)
-		(dnp no)
+		(in_bom no)
+		(on_board yes)
+		(dnp yes)
 		(fields_autoplaced yes)
 		(property "Reference" "IC4"
@@
 		(unit 1)
 		(exclude_from_sim no)
-		(in_bom yes)
-		(on_board yes)
-		(dnp no)
+		(in_bom no)
+		(on_board yes)
+		(dnp yes)
 		(fields_autoplaced yes)
 		(property "Reference" "IC3"
@@
 		(unit 1)
 		(exclude_from_sim no)
-		(in_bom yes)
-		(on_board yes)
-		(dnp no)
+		(in_bom no)
+		(on_board yes)
+		(dnp yes)
 		(fields_autoplaced yes)
 		(property "Reference" "IC2"
@@
 		(unit 1)
 		(exclude_from_sim no)
-		(in_bom yes)
-		(on_board yes)
-		(dnp no)
+		(in_bom no)
+		(on_board yes)
+		(dnp yes)
 		(fields_autoplaced yes)
 		(property "Reference" "IC8"
@@
 		(unit 1)
 		(exclude_from_sim no)
-		(in_bom yes)
-		(on_board yes)
-		(dnp no)
+		(in_bom no)
+		(on_board yes)
+		(dnp yes)
 		(fields_autoplaced yes)
 		(property "Reference" "IC1"
